Commit message: mass:=3 kg

File: src/ur5_description/urdf/ur5_box.urdf.xacro (robot description, xacro)
@@ -355,5 +355,5 @@
     <!-- box  -->
     <xacro:property name="width" value="0.1" />
-    <xacro:property name="mass" value="1" />
+    <xacro:property name="mass" value="3" />
     <link name="box">
       <visual>
